Commit message: improved urdf which was done from weird people, and improved inverse kinematics, added two yaml files, and teleop_send to cobot node and connection teleop_control->inverse_kin->send_to_cobot but speed needs to be gotten and adjusted and also not tested

File: ros2_ws/src/robot_description/urdf/mycobot_280_m5/mycobot_280_m5.urdf (robot description, URDF)
Before this commit: robot firefighter, 8 links, 7 joints
Links:
- removed link g_base
- added link mycobot_base; collision mesh filename=package://robot_description/urdf/mycobot_280_m5/mycobot_bas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; visual mesh filename=package://robot_description/urdf/mycobot_280_m5/mycobot_bas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
Joints:
- removed joint g_base_to_joint1
- added joint mycobot_base_to_joint1: type fixed, parent mycobot_base, child joint1, origin xyz=0 0 0 rpy=0 0 0, axis 0 0 0, limit lower=-3.14 upper=3.14159 effort=1000.0 velocity=0

File: ros2_ws/src/robot_description/urdf/mycobot_280_m5/mycobot_280_m5_adaptive_gripper.urdf (robot description, URDF)
Before this commit: robot firefighter, 15 links, 14 joints
Links:
- removed link g_base
- added link mycobot_base; collision mesh filename=package://robot_description/urdf/mycobot_280_m5/mycobot_bas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; visual mesh filename=package://robot_description/urdf/mycobot_280_m5/mycobot_bas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
Joints:
- removed joint g_base_to_joint1
- added joint mycobot_base_to_joint1: type fixed, parent mycobot_base, child joint1, origin xyz=0 0 0 rpy=0 0 0, axis 0 0 0, limit lower=-3.14 upper=3.14159 effort=1000.0 velocity=0

File: ros2_ws/src/robot_description/urdf/mycobot_280_m5/mycobot_280_m5_camera_adaptive_gripper.urdf (robot description, URDF)
Before this commit: robot firefighter, 16 links, 15 joints
Links:
- removed link camera_flange
- removed link g_base
- removed link joint1
- removed link joint2
- removed link joint3
- removed link joint4
- removed link joint5
- removed link joint6
- removed link joint6_flange
- added link camera; collision mesh filename=package://robot_description/urdf/mycobot_280_m5/camera.dae; visual mesh filename=package://robot_description/urdf/mycobot_280_m5/camera.dae
- added link link1; collision mesh filename=package://robot_description/urdf/mycobot_280_m5/joint1.dae; visual mesh filename=package://robot_description/urdf/mycobot_280_m5/joint1.dae
- added link link2; collision mesh filename=package://robot_description/urdf/mycobot_280_m5/joint2.dae; visual mesh filename=package://robot_description/urdf/mycobot_280_m5/joint2.dae
- added link link3; collision mesh filename=package://robot_description/urdf/mycobot_280_m5/joint3.dae; visual mesh filename=package://robot_description/urdf/mycobot_280_m5/joint3.dae
- added link link4; collision mesh filename=package://robot_description/urdf/mycobot_280_m5/joint4.dae; visual mesh filename=package://robot_description/urdf/mycobot_280_m5/joint4.dae
- added link link5; collision mesh filename=package://robot_description/urdf/mycobot_280_m5/joint5.dae; visual mesh filename=package://robot_description/urdf/mycobot_280_m5/joint5.dae
- added link link6; collision mesh filename=package://robot_description/urdf/mycobot_280_m5/joint6.dae; visual mesh filename=package://robot_description/urdf/mycobot_280_m5/joint6.dae
- added link link7; collision mesh filename=package://robot_description/urdf/mycobot_280_m5/joint7.dae; visual mesh filename=package://robot_description/urdf/mycobot_280_m5/joint7.dae
- added link mycobot_base; collision mesh filename=package://robot_description/urdf/mycobot_280_m5/mycobot_bas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; visual mesh filename=package://robot_description/urdf/mycobot_280_m5/mycobot_bas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
Joints:
- removed joint camera_flange_to_gripper_base
- removed joint g_base_to_joint1
- removed joint joint2_to_joint1
- removed joint joint3_to_joint2
- removed joint joint4_to_joint3
- removed joint joint5_to_joint4
- removed joint joint6_to_joint5
- removed joint joint6output_to_camera_flange
- removed joint joint6output_to_joint6
- added joint base_joint: type fixed, parent mycobot_base, child link1, origin xyz=0 0 0 rpy=0 0 0, axis 0 0 0, limit lower=-3.14 upper=3.14159 effort=1000.0 velocity=0
- added joint camera_to_gripper_base: type fixed, parent camera, child gripper_base, origin xyz=0.0 0.041 0.0 rpy=0 -1.57 0
- added joint joint1: type revolute, parent link1, child link2, origin xyz=0 0 0.13156 rpy=0 0 0, axis 0 0 1, limit lower=-2.9322 upper=2.9322 effort=1000.0 velocity=0
- added joint joint2: type revolute, parent link2, child link3, origin xyz=0 0  0 rpy=0 1.5708 -1.5708, axis 0 0 1, limit lower=-2.3562 upper=2.3562 effort=1000.0 velocity=0
- added joint joint3: type revolute, parent link3, child link4, origin xyz=  -0.1104 0 0    rpy=0 0 0, axis  0 0 1, limit lower=-2.618 upper=2.618 effort=1000.0 velocity=0
- added joint joint4: type revolute, parent link4, child link5, origin xyz=-0.096 0 0.06462 rpy=0 0 -1.5708, axis  0 0 1, limit lower=-2.5307 upper=2.5307 effort=1000.0 velocity=0
- added joint joint5: type revolute, parent link5, child link6, origin xyz=0 -0.07318 0 rpy=1.5708 -1.5708 0, axis 0 0 1, limit lower=-2.8798 upper=2.8798 effort=1000.0 velocity=0
- added joint joint6: type revolute, parent link6, child link7, origin xyz=0 0.0456 0 rpy=-1.5708 0 0, axis 0 0 1, limit lower=-3.14159 upper=3.14159 effort=1000.0 velocity=0
- added joint joint7_to_camera: type fixed, parent link7, child camera, origin xyz=0 0 0.01 rpy=1.579 0 0.7854
- joint gripper_base_to_gripper_left2: origin xyz=-0.005 0.027 0 rpy=0 0 0 -> xyz=-0.005 0.0195 0 rpy=0 0 0
- joint gripper_base_to_gripper_right2: mimic joint=gripper_controller multiplier=-1.0 offset=0 -> joint=gripper_controller multiplier=-1.0 offset=0.0; origin xyz=0.005 0.027 0 rpy=0 0 0 -> xyz=0.005 0.0195 0 rpy=0 0 0
- joint gripper_base_to_gripper_right3: origin xyz=0.012 0.005 0 rpy=0 0 0 -> xyz=0.012 -0.002 0 rpy=0 0 0
- joint gripper_controller: origin xyz=-0.012 0.005 0 rpy=0 0 0 -> xyz=-0.012 -0.002 0 rpy=0 0 0

File: ros2_ws/src/robot_description/urdf/mycobot_280_m5/mycobot_280_m5_with_camera_flange.urdf (robot description, URDF)
Before this commit: robot firefighter, 9 links, 8 joints
Links:
- removed link g_base
- added link mycobot_base; collision mesh filename=package://robot_description/urdf/mycobot_280_m5/mycobot_bas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; visual mesh filename=package://robot_description/urdf/mycobot_280_m5/mycobot_bas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
Joints:
- removed joint g_base_to_joint1
- added joint mycobot_base_to_joint1: type fixed, parent mycobot_base, child joint1, origin xyz=0 0 0 rpy=0 0 0, axis 0 0 0, limit lower=-3.14 upper=3.14159 effort=1000.0 velocity=0

File: ros2_ws/src/robot_description/urdf/mycobot_280_m5/mycobot_280_m5_with_pump.urdf (robot description, URDF)
Before this commit: robot firefighter, 10 links, 9 joints
Links:
- removed link g_base
- added link mycobot_base; collision mesh filename=package://robot_description/urdf/mycobot_280_m5/mycobot_bas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; visual mesh filename=package://robot_description/urdf/mycobot_280_m5/mycobot_bas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
Joints:
- removed joint g_base_to_joint1
- removed joint g_base_to_pump_box
- added joint mycobot_base_to_joint1: type fixed, parent mycobot_base, child joint1, origin xyz=0 0 0 rpy=0 0 0, axis 0 0 0, limit lower=-3.14 upper=3.14159 effort=1000.0 velocity=0
- added joint mycobot_base_to_pump_box: type fixed, parent mycobot_base, child pump_box, origin xyz=0 0 0 rpy=0 0 0, axis 0 0 0, limit lower=-3.14 upper=3.14159 effort=1000.0 velocity=0
