Commit message: wokring wihtout connecting cobot but lagging and also sending to the cobot is ok. Frames are all correct now and basic sturcture

File: ros2_ws/src/robot_description/urdf/mycobot_280_m5/mycobot_280_m5_camera_adaptive_gripper.urdf (robot description, URDF)
Before this commit: robot firefighter, 16 links, 15 joints
Joints:
- joint joint7_to_camera: origin xyz=0 0 0.01 rpy=1.579 0 0.7854 -> xyz=0 0 0.01 rpy=1.579 0 -2.3562

Commit message: WOrking good! Visualization of frames in mujoco, updated tf speed and urdf correcting, added block to grasp in xml but friction and collision not so good

File: ros2_ws/src/robot_description/urdf/mycobot_280_m5/mycobot_280_m5_camera_adaptive_gripper.urdf (robot description, URDF)
Before this commit: robot firefighter, 16 links, 15 joints
Joints:
- joint base_joint: origin xyz=0 0 0 rpy=0 0 0 -> xyz=0 0 0.032 rpy=0 0 0

Commit message: NOW WOKRING GOOD! Camera and audio seperate thread, improved camera settings, added LED status of mycobot, changed xmla dn urdf and static tf to move base lower liek real robot, improved other settings.

File: ros2_ws/src/robot_description/urdf/mycobot_280_m5/mycobot_280_m5_camera_adaptive_gripper.urdf (robot description, URDF)
Before this commit: robot firefighter, 16 links, 15 joints
Joints:
- joint base_joint: origin xyz=0 0 0.032 rpy=0 0 0 -> xyz=0 0 0.0 rpy=0 0 0

Commit message: rgb point cloud with accumulating points wokring and cut off botom of image but tf in urdf and mujoco not matching

File: ros2_ws/src/robot_description/urdf/mycobot_280_m5/mycobot_280_m5_camera_adaptive_gripper.urdf (robot description, URDF)
Before this commit: robot firefighter, 16 links, 15 joints
Links:
- added link camera_lens
Joints:
- added joint camera_to_camera_lens: type fixed, parent camera, child camera_lens, origin xyz=0.042 0.005 0 rpy=-1.5708 1.5708 -0.1
